File: 50_Shot_Relay_V0.0.sch (EAGLE design)
At the start: 183 parts, among them J1 J13, J2 J14, J3 J15, J4 J16, Q1 Qs5U34CT-ND, Q10 Qs5U34CT-ND, Q11 Qs5U34CT-ND, Q12 Qs5U34CT-ND, Q13 Qs5U34CT-ND, Q14 Qs5U34CT-ND, Q15 Qs5U34CT-ND, Q16 Qs5U34CT-ND, Q17 Qs5U34CT-ND, Q18 Qs5U34CT-ND, Q19 Qs5U34CT-ND, Q2 Qs5U34CT-ND, Q20 Qs5U34CT-ND, Q21 Qs5U34CT-ND, Q22 Qs5U34CT-ND, Q23 Qs5U34CT-ND, Q24 Qs5U34CT-ND, Q25 Qs5U34CT-ND, Q26 Qs5U34CT-ND, Q27 Qs5U34CT-ND, Q28 Qs5U34CT-ND, Q29 Qs5U34CT-ND, Q3 Qs5U34CT-ND, Q30 Qs5U34CT-ND, Q4 Qs5U34CT-ND, Q5 Qs5U34CT-ND, Q6 Qs5U34CT-ND, Q7 Qs5U34CT-ND, Q8 Qs5U34CT-ND, Q9 Qs5U34CT-ND, U1 MM74HC595, U2 MM74HC595, U3 7400, U4 MM74HC245, U5 MM74HC245, U6 ULN2803ADW, U7 ULN2803ADW, X1 22-23-2111, X2 22-23-2111, X3 22-23-2091, X4 22-23-2031, X5 22-23-2101, X6 22-23-2101

Commit message: add proper relay board
Parts:
- removed C6: 0.01uF, rcl:C-USC0805
- removed D18, D19, D20: 5.0V, Mine:568-6471-1-ND_ZENER_5.0V
- removed D21: SA2M-E3/5ATGICT-ND, Mine:DIODE_SA2M-E3/5ATGICT-ND
- removed J1: J13, Mine:22-23-2061
- removed J2: J14, Mine:22-23-2061
- removed J3: J15, Mine:22-23-2061
- removed J4: J16, Mine:22-23-2061
- removed Q25, Q26, Q27, Q28, Q29, Q30: Qs5U34CT-ND, Mine:QS5U34CT-ND_MOSFET_N_CHANNEL
- removed R75: 1M, rcl:R-US_M0805
- removed R76, R77, R78, R88, R89, R90: 1k, rcl:R-US_M0805
- removed R79, R80, R81, R85, R86, R87: 100k, rcl:R-US_M0805
- removed R82, R83, R84: 10k, rcl:R-US_M0805
- removed RLY17, RLY18, RLY19, RLY20: OMRON, Mine:OMRON
- removed U5: MM74HC245, Mine:MM74HC245
- removed U6, U7: ULN2803ADW, Texas Instruments_By_element14_Batch_1:ULN2803ADW
- added LED1, LED2: LEDCHIP-LED0805, Mine:LEDCHIP-LED0805
- added X7: 22-23-2091, Mine:22-23-2091
- added X8, X9: 22-23-2081, Mine:22-23-2081
- C1: value .01uf -> 0.01uF; MPN 103GCR050M -> VY2103M63Y5US63V7; OC_NEWARK 02P3403 -> 69K4077
- C2: MPN (none) -> VY2103M63Y5US63V7; OC_NEWARK unknown -> 69K4077
- D1, D10, D11, D2, D3, D4, D5: value SA2M-E3/5ATGICT-ND -> 5.0V; device Mine:DIODE_SA2M-E3/5ATGICT-ND -> Mine:568-6471-1-ND_ZENER_5.0V
- D13, D14, D15, D7, D8, D9: value 5.0V -> SA2M-E3/5ATGICT-ND; device Mine:568-6471-1-ND_ZENER_5.0V -> Mine:DIODE_SA2M-E3/5ATGICT-ND
- R1, R2: value 330 -> 100
- R10: value 560 -> 1k
- R11, R28: value 10k -> 330
- R12, R45, R60, R68: value 10k -> 100k
- R14, R20, R23, R24: value 100k -> 330
- R15, R16: value 1M -> 10k
- R17, R25: value 1k -> 330
- R18, R52, R64, R66: value 1k -> 100k
- R21, R22, R58, R69: value 10k -> 1k
- R26, R53, R54, R65: value 1k -> 10k
- R3, R4: value 330 -> 10k
- R47, R48, R61: value 100k -> 1M
- R49, R50, R74: value 1M -> 1k
- R5, R6: value 330 -> 100k
- R51, R73: value 1M -> 100k
- R57, R63, R70: value 100k -> 1k
- R62, R72: value 100k -> 10k
- R67: value 10k -> 1M
- R7: value 330 -> 1M
- R8: value 560 -> 1M
- R9: value 330 -> 1k
- U2: value MM74HC595 -> 7400; device Mine:MM74HC595 -> 74xx-us:7400
- U3: value 7400 -> MM74HC245; device 74xx-us:7400 -> Mine:MM74HC245
- U4: value MM74HC245 -> ULN2803ADW; device Mine:MM74HC245 -> Texas Instruments_By_element14_Batch_1:ULN2803ADW; MF (none) -> TEXAS INSTRUMENTS; OC_NEWARK unknown -> (none)
- X1, X2: OC_NEWARK (none) -> unknown
- X3: value 22-23-2091 -> 22-23-2051; device Mine:22-23-2091 -> Mine:22-23-2051
- X4: value 22-23-2031 -> 22-23-2051; device Mine:22-23-2031 -> Mine:22-23-2051
- X5, X6: value 22-23-2101 -> 22-23-2051; device con-molex:22-23-2101 -> Mine:22-23-2051
Connections:
- removed net CH10_A: RLY162.P, X6-9.S
- removed net CH10_B: RLY163.P, X6-10.S
- removed net CH9_A: RLY202.P, X6-7.S
- removed net CH9_B: RLY203.P, X6-8.S
- removed net GLV10_GRN: J2-5.S, R78.1
- removed net GLV10_RED: J4-5.S, R90.1
- removed net GLV9_GRN: J2-4.S, R77.1
- removed net GLV9_RED: J4-4.S, R89.1
- removed net GLV_10: R69.2, RLY163.S
- removed net GLV_9: R68.2, RLY203.S
- removed net N$101: RLY182.S, RLY183.P, RLY202.O
- removed net N$162: D19.C, Q26.G, R68.1, R71.2, R80.2
- removed net N$163: Q23.G, R71.1, R74.2
- removed net N$164: Q23.S, R74.1, R77.2
- removed net N$165: Q26.D, Q29.G, R83.1, R86.2
- removed net N$166: Q29.S, R86.1, R89.2
- removed net N$169: D20.C, Q27.G, R69.1, R72.2, R81.2
- removed net N$170: Q24.G, R72.1, R75.2
- removed net N$171: Q24.S, R75.1, R78.2
- removed net N$172: Q27.D, Q30.G, R84.1, R87.2
- removed net N$173: Q30.S, R87.1, R90.2
- removed net N$179: R3.1, X3-6.S
- removed net N$180: R2.1, X3-7.S
- removed net N$181: R1.1, X3-8.S
- removed net N$182: R10.1, X4-1.S
- removed net N$183: R8.1, X4-2.S
- removed net N$19: R10.2, U2.QA, U5.A1
- removed net N$20: R8.2, U2.QB, U5.A2
- removed net N$21: U1.QH*, U2.SER
- removed net N$22: U2.QC, U5.A3
- removed net N$23: U2.QD, U5.A4
- removed net N$24: U2.QE, U5.A5
- removed net N$25: U2.QF, U5.A6
- removed net N$26: U2.QG, U5.A7
- removed net N$27: U2.QH, U5.A8
- removed net N$35: U5.B1, U7.1B
- removed net N$36: U5.B2, U7.2B
- removed net N$37: U5.B3, U7.3B
- removed net N$38: U5.B4, U7.4B
- removed net N$39: U5.B5, U7.5B
- removed net N$40: U5.B6, U7.6B
- removed net N$41: U5.B7, U7.7B
- removed net N$42: U5.B8, U7.8B
- removed net N$44: U3B.O, U5.OE
- removed net N$52: RLY181.-, U7.1C
- removed net N$53: RLY131.-, U7.2C
- removed net N$54: X1-8.S
- removed net N$55: X1-9.S
- removed net N$56: X1-10.S
- removed net N$57: X1-11.S
- removed net N$7: X1-6.S
- removed net N$8: X1-7.S
- removed net N$91: RLY132.S, RLY133.P, RLY162.O
- new net QN_ALT: U1.QH*, X2-9.S
- net ARM_RELAY: now also RLY151.+, U4.COM, X1-7.S, X2-5.S; no longer RLY131.+, RLY171.+, RLY181.+, U6.COM, U7.COM, X2-7.S
- net CH1_A: now also X8-1.S; no longer X5-1.S
- net CH1_B: now also X8-2.S; no longer X5-2.S
- net CH2_A: now also X8-3.S; no longer X5-3.S
- net CH2_B: now also X8-4.S; no longer X5-4.S
- net CH3_A: now also X8-5.S; no longer X5-5.S
- net CH3_B: now also X8-6.S; no longer X5-6.S
- net CH4_A: now also X8-7.S; no longer X5-7.S
- net CH4_B: now also X8-8.S; no longer X5-8.S
- net CH5_A: now also X9-1.S; no longer X5-9.S
- net CH5_B: now also X9-2.S; no longer X5-10.S
- net CH6_A: now also RLY132.P, X9-3.S; no longer RLY142.P, X6-1.S
- net CH6_B: now also RLY133.P, X9-4.S; no longer RLY143.P, X6-2.S
- net CH7_A: now also RLY162.P, X9-5.S; no longer RLY192.P, X6-3.S
- net CH7_B: now also RLY163.P, X9-6.S; no longer RLY193.P, X6-4.S
- net CH8_A: now also RLY142.P, X9-7.S; no longer RLY152.P, X6-5.S
- net CH8_B: now also RLY143.P, X9-8.S; no longer RLY153.P, X6-6.S
- net F_BATT: now also RLY152.P, X1-10.S, X2-2.S; no longer RLY132.P, RLY172.P, RLY182.P, X2-10.S
- net GLV1_GRN: now also R9.1, X3-1.S; no longer J1-1.S, R17.1
- net GLV1_RED: now also R21.1, X5-1.S; no longer J3-1.S, R25.1
- net GLV2_GRN: now also R10.1, X3-2.S; no longer J1-2.S, R18.1
- net GLV2_RED: now also R22.1, X5-2.S; no longer J3-2.S, R26.1
- net GLV3_GRN: now also X3-3.S; no longer J1-3.S
- net GLV3_RED: now also X5-3.S; no longer J3-3.S
- net GLV4_GRN: now also X3-4.S; no longer J1-4.S
- net GLV4_RED: now also X5-4.S; no longer J3-4.S
- net GLV5_GRN: now also R49.1, X4-1.S; no longer J1-5.S, R52.1
- net GLV5_RED: now also R57.1, X6-1.S; no longer J3-5.S, R64.1
- net GLV6_GRN: now also R50.1, X4-2.S; no longer J2-1.S, R53.1
- net GLV6_RED: now also R58.1, X6-2.S; no longer J4-1.S, R65.1
- net GLV7_GRN: now also R63.1, X4-3.S; no longer J2-2.S, R54.1
- net GLV7_RED: now also R70.1, X6-3.S; no longer J4-2.S, R66.1
- net GLV8_GRN: now also R69.1, X4-4.S; no longer J2-3.S, R76.1
- net GLV8_RED: now also R74.1, X6-4.S; no longer J4-3.S, R88.1
- net GLV_1: now also R3.2; no longer R11.2
- net GLV_2: now also R4.2; no longer R12.2
- net GLV_3: now also R26.2; no longer R27.2
- net GLV_4: now also R27.2; no longer R28.2
- net GLV_6: now also RLY133.S; no longer RLY143.S
- net GLV_7: now also R59.2, RLY163.S; no longer R45.2, RLY193.S
- net GLV_8: now also R62.2, RLY143.S; no longer R67.2, RLY153.S
- net GLV_PB: now also Q17.D, Q18.D, R15.2, R16.2, R53.2, R54.2, R65.2, R72.2, X1-11.S, X2-1.S; no longer Q15.D, Q20.D, Q23.D, Q28.D, Q29.D, Q30.D, R21.2, R22.2, R58.2, R59.2, R60.2, R82.2, R83.2, R84.2, X2-11.S
- net GLV_RELAY: now also X1-8.S, X2-4.S; no longer X2-8.S
- net GLV_SW: now also D13.C, D14.C, D15.C, D7.C, D8.C, D9.C, RLY131.+, RLY132.S, X1-9.S, X2-3.S; no longer D1.C, D10.C, D11.C, D2.C, D21.C, D3.C, D4.C, D5.C, RLY151.+, RLY152.S, RLY191.+, RLY192.S, RLY201.+, RLY202.S, X2-9.S
- net GND: now also LED1.C, LED2.C, Q15.S, Q20.S, Q23.S, R12.1, R13.1, R51.1, R52.1, R64.1, R71.1, RLY131.-, U2B.I0, U2B.I1, U2C.I0, U2C.I1, U2D.I0, U2D.I1, U2P.GND, U3.GND, X1-2.S, X2-10.S, X3-5.S, X4-5.S, X5-5.S, X6-5.S, X7-1.S; no longer C6.2, D18.A, D19.A, D20.A, D21.A, J1-6.S, J2-6.S, J3-6.S, J4-6.S, Q17.S, Q18.S, Q25.S, Q26.S, Q27.S, R19.1, R20.1, R55.1, R56.1, R57.1, R79.1, R80.1, R81.1, RLY151.-, RLY173.O, RLY183.O, RLY191.-, RLY193.O, RLY201.-, RLY203.O, U2.G, U2.GND, U3C.I0, U3C.I1, U3D.I0, U3D.I1, U3P.GND, U5.GND, U6.GND, U7.GND, X2-2.S, X3-9.S, X4-3.S
- net N$1: now also LED2.A, R2.1; no longer X1-1.S
- net N$10: now also R25.2, U3.A2; no longer R7.2, U4.A2
- net N$106: now also D1.C, R12.2, R3.1, R5.2; no longer D6.C, R11.1, R13.2, R19.2
- net N$107: now also R5.1, R7.2; no longer R13.1, R15.2
- net N$108: now also R18.1, R21.2; no longer R23.1, R25.2
- net N$109: now also R7.1, R9.2; no longer R15.1, R17.2
- net N$11: now also R24.2, U3.A3; no longer R6.2, U4.A3
- net N$110: now also R15.1, R18.2; no longer R21.1, R23.2
- net N$114: now also D2.C, R13.2, R4.1, R6.2; no longer D7.C, R12.1, R14.2, R20.2
- net N$115: now also R6.1, R8.2; no longer R14.1, R16.2
- net N$116: now also R10.2, R8.1; no longer R16.1, R18.2
- net N$117: now also R16.1, R19.2; no longer R22.1, R24.2
- net N$118: now also R19.1, R22.2; no longer R24.1, R26.2
- net N$12: now also R23.2, U3.A4; no longer R5.2, U4.A4
- net N$120: now also D3.C, R26.1; no longer D8.C, R27.1
- net N$127: now also D4.C, R27.1; no longer D9.C, R28.1
- net N$13: now also R20.2, U3.A5; no longer R4.2, U4.A5
- net N$134: now also D10.C, Q20.G, R59.1, R60.2, R64.2; no longer D15.C, Q18.G, R45.1, R48.2, R57.2
- net N$135: now also Q19.G, R60.1, R61.2; no longer Q15.G, R48.1, R51.2
- net N$136: now also Q19.S, R61.1, R63.2; no longer Q15.S, R51.1, R54.2
- net N$137: now also Q20.D, Q22.G, R65.1, R68.2; no longer Q18.D, Q21.G, R60.1, R63.2
- net N$138: now also Q22.S, R68.1, R70.2; no longer Q21.S, R63.1, R66.2
- net N$14: now also R17.2, U3.A6; no longer R3.2, U4.A6
- net N$141: now also D6.C, Q16.G, R46.2, R52.2; no longer D14.C, Q17.G, R47.2, R56.2
- net N$142: now also R46.1, R48.2; no longer R47.1, R50.2
- net N$143: now also R48.1, R50.2; no longer R50.1, R53.2
- net N$144: now also Q16.D, Q18.G, R54.1, R56.2; no longer Q17.D, Q20.G, R59.1, R62.2
- net N$145: now also Q18.S, R56.1, R58.2; no longer Q20.S, R62.1, R65.2
- net N$148: now also D5.C, Q15.G, R45.2, R51.2; no longer D13.C, Q16.G, R46.2, R55.2
- net N$149: now also R45.1, R47.2; no longer R46.1, R49.2
- net N$15: now also R14.2, U3.A7; no longer R2.2, U4.A7
- net N$150: now also R47.1, R49.2; no longer R49.1, R52.2
- net N$151: now also Q15.D, Q17.G, R53.1, R55.2; no longer Q16.D, Q19.G, R58.1, R61.2
- net N$152: now also Q17.S, R55.1, R57.2; no longer Q19.S, R61.1, R64.2
- net N$155: now also D11.C, Q23.G, R62.1, R66.2, R71.2; no longer D18.C, Q25.G, R67.1, R70.2, R79.2
- net N$156: now also Q21.G, R66.1, R67.2; no longer Q22.G, R70.1, R73.2
- net N$157: now also Q21.S, R67.1, R69.2; no longer Q22.S, R73.1, R76.2
- net N$158: now also Q23.D, Q24.G, R72.1, R73.2; no longer Q25.D, Q28.G, R82.1, R85.2
- net N$159: now also Q24.S, R73.1, R74.2; no longer Q28.S, R85.1, R88.2
- net N$16: now also R11.2, U3.A8; no longer R1.2, U4.A8
- net N$17: now also U3.B1, U4.1B; no longer U4.B1, U6.1B
- net N$174: now also R28.1, X7-9.S; no longer R9.1, X3-1.S
- net N$175: now also R25.1, X7-8.S; no longer R7.1, X3-2.S
- net N$176: now also R24.1, X7-7.S; no longer R6.1, X3-3.S
- net N$177: now also R23.1, X7-6.S; no longer R5.1, X3-4.S
- net N$178: now also R20.1, X7-5.S; no longer R4.1, X3-5.S
- net N$18: now also U2A.O, U3.OE; no longer U3A.O, U4.OE
- net N$2: now also R17.1, X7-4.S; no longer X1-2.S
- net N$28: now also U3.B2, U4.2B; no longer U4.B2, U6.2B
- net N$29: now also U3.B3, U4.3B; no longer U4.B3, U6.3B
- net N$3: now also R14.1, X7-3.S; no longer X1-3.S
- net N$30: now also U3.B4, U4.4B; no longer U4.B4, U6.4B
- net N$31: now also U3.B5, U4.5B; no longer U4.B5, U6.5B
- net N$32: now also U3.B6, U4.6B; no longer U4.B6, U6.6B
- net N$33: now also U3.B7, U4.7B; no longer U4.B7, U6.7B
- net N$34: now also U3.B8, U4.8B; no longer U4.B8, U6.8B
- net N$4: now also LED1.A, R1.2; no longer X1-4.S
- net N$43: now also U4.1C; no longer U6.1C
- net N$45: now also U4.2C; no longer U6.2C
- net N$46: now also U4.3C; no longer U6.3C
- net N$47: now also U4.4C; no longer U6.4C
- net N$48: now also U4.5C; no longer U6.5C
- net N$49: now also U4.6C; no longer U6.6C
- net N$5: now also R11.1, X7-2.S; no longer X1-5.S
- net N$50: now also RLY151.-, U4.7C; no longer RLY171.-, U6.7C
- net N$51: now also U4.8C; no longer U6.8C
- net N$80: now also RLY132.O; no longer RLY142.O
- net N$87: now also RLY142.O; no longer RLY152.O
- net N$9: now also R28.2, U3.A1; no longer R9.2, U4.A1
- net N$94: now also RLY152.S, RLY153.P, RLY162.O; no longer RLY172.S, RLY173.P, RLY192.O
- net RCLK: now also X1-6.S; no longer U2.RCLK
- net SER: now also X1-3.S; no longer X2-3.S
- net SRCLK: now also U2A.I0, U2A.I1, X1-4.S, X2-8.S; no longer U2.SRCLK, U3A.I0, U3A.I1, U3B.I0, U3B.I1, X2-4.S
- net SRCLR: now also X1-5.S, X2-7.S; no longer U2.SCLR, X2-5.S
- net VDD: now also R1.1, R2.2, U2P.VCC, U3.DIR, U3.VCC, X1-1.S, X2-11.S; no longer C6.1, U2.VCC, U3P.VCC, U4.DIR, U4.VCC, U5.DIR, U5.VCC, X2-1.S
Other:
- note added: "GREEN"
- note added: "RED"
- note added: "Return Header"
- note removed: "Added this file"
- moved on the sheet: C1, C2, C3, C4, C5, D12, D16, D6, Q1, Q10, Q11, Q12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
