File: 50_Shot_CPU_V0.0.brd (EAGLE design)
At the start: 86 x 100 mm, 75 parts, among them IC1 PIC24FJ128GA010, IC2 93LC46ST, J1 J12, J12 A311422_nd, J13 22-23-2021, J14 22-23-2021, J3 22-23-2021, J4 22-23-2021, J5 22-23-2021, Q1 Qs5U34CT-ND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

Commit message: Added fire/reset/encoder switches
Parts:
- removed J3, J4, J5: 22-23-2021, Mine:22-23-2021
- added JP15, JP16, JP17: SHERLOCK_2PIN_RGT, Mine:SHERLOCK_2PIN_RGT
Connections:
- net GND: now also JP17.2; no longer J5.2
- net N$58: now also JP15.2; no longer J3.2
- net N$7: now also JP17.1; no longer J5.1
- net N$8: now also JP16.2; no longer J4.2
- net VDD: now also JP15.1, JP16.1; no longer J3.1, J4.1
Routing:
- net VDD: track 377.5 -> 365.6 mm
- net N$58: track 73.4 -> 64.5 mm
- net N$7: track 25.9 -> 24.4 mm
- net N$8: track 22.3 -> 20.8 mm
Other:
- board text added: "Fire_ SW"
- board text added: "Parallel A"
- board text added: "Parallel B"
- board text added: "RST_ SW"
- board text added: "UART"
Changed lines of the file:
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@@
 <text x="1.27" y="-41.91" size="1.016" layer="21">Rotary
 Encoder</text>
-<text x="3.048" y="-56.134" size="1.016" layer="21">I2C Header</text>
+<text x="45.974" y="-46.482" size="1.016" layer="21">I2C Header</text>
 <text x="1.27" y="-72.644" size="1.016" layer="21">Expansion
    B</text>
@@
 <text x="76.708" y="-13.462" size="1.016" layer="21">ON_
 LED</text>
+<text x="4.318" y="-101.854" size="1.016" layer="21">Parallel A</text>
+<text x="3.81" y="-117.602" size="1.016" layer="21">Parallel B</text>
+<text x="4.572" y="-131.064" size="1.016" layer="21">UART</text>
+<text x="1.524" y="-147.32" size="1.016" layer="21">Fire_
+SW</text>
+<text x="13.208" y="-146.558" size="1.016" layer="21">RST_
+SW</text>
 </plain>
 <attributes>
@@
 <attribute name="NAME" x="6.985" y="94.352" size="1.778" layer="25" rot="R180"/>
 </element>
-<element name="J3" library="Mine" package="22-23-2021" value="22-23-2021" x="4.93" y="72.314" smashed="yes" rot="R90">
-<attribute name="MPN" value="22-23-2021" x="4.93" y="72.314" size="1.778" layer="27" rot="R90" display="off"/>
-<attribute name="OC_FARNELL" value="1462926" x="4.93" y="72.314" size="1.778" layer="27" rot="R90" display="off"/>
-<attribute name="MF" value="MOLEX" x="4.93" y="72.314" size="1.778" layer="27" rot="R90" display="off"/>
-<attribute name="OC_NEWARK" value="25C3832" x="4.93" y="72.314" size="1.778" layer="27" rot="R90" display="off"/>
-<attribute name="NAME" x="3.378" y="68.938" size="1.27" layer="25" ratio="10" rot="R180"/>
-</element>
-<element name="J4" library="Mine" package="22-23-2021" value="22-23-2021" x="5.93" y="20.9" smashed="yes" rot="R90">
-<attribute name="MPN" value="22-23-2021" x="5.93" y="20.9" size="1.778" layer="27" rot="R90" display="off"/>
-<attribute name="OC_FARNELL" value="1462926" x="5.93" y="20.9" size="1.778" layer="27" rot="R90" display="off"/>
-<attribute name="MF" value="MOLEX" x="5.93" y="20.9" size="1.778" layer="27" rot="R90" display="off"/>
-<attribute name="OC_NEWARK" value="25C3832" x="5.93" y="20.9" size="1.778" layer="27" rot="R90" display="off"/>
-<attribute name="NAME" x="11.358" y="23.456" size="1.016" layer="25" ratio="10" rot="R180"/>
-</element>
-<element name="J5" library="Mine" package="22-23-2021" value="22-23-2021" x="5.93" y="14.772" smashed="yes" rot="R90">
-<attribute name="MPN" value="22-23-2021" x="5.93" y="14.772" size="1.778" layer="27" rot="R90" display="off"/>
-<attribute name="OC_FARNELL" value="1462926" x="5.93" y="14.772" size="1.778" layer="27" rot="R90" display="off"/>
-<attribute name="MF" value="MOLEX" x="5.93" y="14.772" size="1.778" layer="27" rot="R90" display="off"/>
-<attribute name="OC_NEWARK" value="25C3832" x="5.93" y="14.772" size="1.778" layer="27" rot="R90" display="off"/>
-<attribute name="NAME" x="11.39" y="17.36" size="1.016" layer="25" ratio="10" rot="R180"/>
-</element>
 <element name="Q1" library="Mine" package="SOT23-5L" value="Qs5U34CT-ND" x="49.47" y="78.99" smashed="yes" rot="R270">
 <attribute name="NAME" x="47.883" y="81.093" size="1.27" layer="25"/>
@@
 <element name="JP13" library="Mine" package="SHERLOCK_8PIN-RGT" value="SHERLOCK_8PIN_RGT" x="8.89" y="-123.19"/>
 <element name="JP14" library="Mine" package="SHERLOCK_6PIN_RGT" value="SHERLOCK_6PIN_RGT" x="7.112" y="-136.398"/>
+<element name="JP15" library="Mine" package="SHERLOCK_2PIN_RGT" value="SHERLOCK_2PIN_RGT" x="2.032" y="-151.638"/>
+<element name="JP16" library="Mine" package="SHERLOCK_2PIN_RGT" value="SHERLOCK_2PIN_RGT" x="13.716" y="-151.384"/>
+<element name="JP17" library="Mine" package="SHERLOCK_2PIN_RGT" value="SHERLOCK_2PIN_RGT" x="2.032" y="-166.878"/>
 </elements>
 <signals>
@@
 <contactref element="C5" pad="2"/>
 <contactref element="R12" pad="1"/>
-<contactref element="J5" pad="2"/>
 <contactref element="R11" pad="1"/>
 <contactref element="U1" pad="10"/>
@@
 <contactref element="JP12" pad="1"/>
 <contactref element="JP14" pad="2"/>
+<contactref element="JP17" pad="2"/>
+<wire x1="10.112" y1="-136.398" x2="2.032" y2="-166.878" width="0" layer="19" extent="1-1"/>
 <wire x1="15.89" y1="-107.95" x2="10.112" y2="-136.398" width="0" layer="19" extent="1-1"/>
 <wire x1="2.064" y1="-46.99" x2="15.89" y2="-107.95" width="0" layer="19" extent="1-1"/>
@@
 <contactref element="U1" pad="20"/>
 <contactref element="C5" pad="1"/>
-<contactref element="J4" pad="1"/>
-<contactref element="J3" pad="1"/>
 <contactref element="J12" pad="5"/>
 <contactref element="R3" pad="2"/>
@@
 <wire x1="32.29" y1="66.58" x2="32.29" y2="67.64" width="0.254" layer="1"/>
 <wire x1="26.924" y1="61.214" x2="32.29" y2="66.58" width="0.254" layer="1"/>
-<wire x1="4.93" y1="71.044" x2="4.93" y2="66.952" width="0.254" layer="16"/>
-<wire x1="4.93" y1="66.952" x2="5.842" y2="66.04" width="0.254" layer="16"/>
-<wire x1="5.842" y1="66.04" x2="5.842" y2="63.212" width="0.254" layer="16"/>
 <wire x1="21.59" y1="36.83" x2="21.59" y2="36.576" width="0.254" layer="1"/>
 <wire x1="21.59" y1="36.576" x2="20.574" y2="35.56" width="0.254" layer="1"/>
@@
 <wire x1="12.192" y1="19.558" x2="9.652" y2="19.558" width="0.254" layer="16"/>
 <wire x1="9.652" y1="19.558" x2="9.58" y2="19.63" width="0.254" layer="16"/>
-<wire x1="9.58" y1="19.63" x2="5.93" y2="19.63" width="0.254" layer="16"/>
 <wire x1="9.906" y1="17.526" x2="9.652" y2="17.78" width="0.254" layer="16"/>
 <wire x1="9.652" y1="17.78" x2="9.652" y2="19.558" width="0.254" layer="16"/>
@@
 <contactref element="JP12" pad="2"/>
 <contactref element="JP14" pad="1"/>
+<contactref element="JP15" pad="1"/>
+<contactref element="JP16" pad="1"/>
+<wire x1="4.032" y1="-151.638" x2="15.716" y2="-151.384" width="0" layer="19" extent="1-1"/>
+<wire x1="12.112" y1="-136.398" x2="4.032" y2="-151.638" width="0" layer="19" extent="1-1"/>
 <wire x1="13.89" y1="-107.95" x2="12.112" y2="-136.398" width="0" layer="19" extent="1-1"/>
 <wire x1="43.546" y1="-51.308" x2="13.89" y2="-107.95" width="0" layer="19" extent="1-1"/>
@@
 <wire x1="32.31" y1="72.33" x2="32.29" y2="72.31" width="0" layer="19" extent="1-1"/>
 <wire x1="54.356" y1="24.13" x2="53.5194" y2="21.4106" width="0" layer="19" extent="1-1"/>
-<wire x1="5.842" y1="63.212" x2="10.414" y2="63.754" width="0" layer="19" extent="1-16"/>
 <wire x1="-1.59" y1="-9.144" x2="15.756" y2="7.052" width="0" layer="19" extent="1-1"/>
 </signal>
@@
 </signal>
 <signal name="N$8">
-<contactref element="J4" pad="2"/>
 <contactref element="R12" pad="2"/>
 <contactref element="U1" pad="5"/>
@@
 <wire x1="8.382" y1="26.924" x2="8.382" y2="23.114" width="0.254" layer="16"/>
 <wire x1="8.382" y1="23.114" x2="7.438" y2="22.17" width="0.254" layer="16"/>
-<wire x1="7.438" y1="22.17" x2="5.93" y2="22.17" width="0.254" layer="16"/>
 <wire x1="17.1098" y1="26.5444" x2="17.272" y2="26.7066" width="0.254" layer="1"/>
 <wire x1="17.272" y1="26.7066" x2="17.272" y2="28.041" width="0.254" layer="1"/>
+<contactref element="JP16" pad="2"/>
+<wire x1="7.438" y1="22.17" x2="13.716" y2="-151.384" width="0" layer="19" extent="16-16"/>
 </signal>
 <signal name="ARM_LED">
@@
 </signal>
 <signal name="N$7">
-<contactref element="J5" pad="1"/>
 <contactref element="U1" pad="6"/>
 <wire x1="22.035" y1="27.391" x2="21.041" y2="27.391" width="0.254" layer="1"/>
@@
 <wire x1="20.32" y1="22.352" x2="20.32" y2="21.59" width="0.254" layer="1"/>
 <wire x1="20.32" y1="21.59" x2="17.018" y2="18.288" width="0.254" layer="1"/>
-<wire x1="5.97" y1="13.462" x2="5.93" y2="13.502" width="0.254" layer="1"/>
 <wire x1="17.018" y1="18.288" x2="10.414" y2="18.288" width="0.254" layer="1"/>
 <wire x1="10.414" y1="18.288" x2="8.636" y2="16.51" width="0.254" layer="1"/>
 <wire x1="8.636" y1="16.51" x2="8.636" y2="14.732" width="0.254" layer="1"/>
 <wire x1="8.636" y1="14.732" x2="7.406" y2="13.502" width="0.254" layer="1"/>
-<wire x1="7.406" y1="13.502" x2="5.93" y2="13.502" width="0.254" layer="1"/>
+<contactref element="JP17" pad="1"/>
+<wire x1="7.406" y1="13.502" x2="4.032" y2="-166.878" width="0" layer="19" extent="1-1"/>
 </signal>
 <signal name="ENCDR_SW">
@@
 </signal>
 <signal name="N$58">
-<contactref element="J3" pad="2"/>
 <contactref element="U1" pad="4"/>
 <contactref element="R11" pad="2"/>
@@
 <wire x1="2.032" y1="31.242" x2="2.032" y2="72.39" width="0.254" layer="1"/>
 <wire x1="2.032" y1="72.39" x2="3.226" y2="73.584" width="0.254" layer="1"/>
-<wire x1="3.226" y1="73.584" x2="4.93" y2="73.584" width="0.254" layer="1"/>
-<wire x1="4.93" y1="73.584" x2="12.184" y2="73.584" width="0.254" layer="1"/>
 <wire x1="12.184" y1="73.584" x2="12.302" y2="73.466" width="0.254" layer="1"/>
+<contactref element="JP15" pad="2"/>
+<wire x1="8.636" y1="28.194" x2="2.032" y2="-151.638" width="0" layer="19" extent="1-1"/>
+<wire x1="12.184" y1="73.584" x2="3.226" y2="73.584" width="0" layer="19" extent="1-1"/>
 </signal>
 <signal name="F_BATT">
